File: Bull Space_ Des by Sheenyl Hassan.kicad_sch (KiCad schematic)
At the start: 17 parts, among them IC1 TEENSY_4.0, IC2 XB24CZ7PIT-004, J1 Screw_Terminal_01x02, J2 Screw_Terminal_01x02, U1 Regulator_Linear_AP2204RB-3.3, U2 Flight-Computer_Adafruit_GPS_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, U3 ADXL343, U4 BMP280, U6 Memory_Flash_W25Q32JVSS

Commit message: Add files via upload
Parts:
- C2: value 47pf -> 1uf
- C4: value 1uf -> 47pf
Connections:
- net +3V3: now also IC1.16 (3.3V)
- net ADXL-CS: now also IC1.12 (10); no longer IC1.11 (9)
- net BMP-CS: now also IC1.11 (9); no longer IC1.10 (8)
- net FL-CS: now also IC1.10 (8); no longer IC1.12 (10)
- net GND: now also BZ1.2 (+)
- net MISO: now also U3.12 (SDO/ADDR), U4.5 (SDO); no longer U3.13 (SDA/SDI/SDIO), U4.3 (SDI)
- net MOSI: now also U3.13 (SDA/SDI/SDIO), U4.3 (SDI); no longer U3.12 (SDO/ADDR), U4.5 (SDO)
- net XBEE-RX: now also IC2.3 (DIN/~{CONFIG}); no longer IC2.2 (DOUT)
- net XBEE-TX: now also IC2.2 (DOUT); no longer IC2.3 (DIN/~{CONFIG})
- no-connect marks 45 -> 44
Other:
- moved on the sheet: BZ1, C1, C2, C4, C5, D1, IC1, IC2, J1, J2, U1, U2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

Commit message: Updates
Parts:
- added R2, R3, R4: 220, Resistor_SMD:R_0603_1608Metric_Pad0.98x0.95mm_HandSolder, symbol Device:R
- C1, C5: footprint Capacitor_SMD:C_0603_1608Metric_Pad1.08x0.95mm_HandSolder -> Capacitor_SMD:C_0805_2012Metric_Pad1.18x1.45mm_HandSolder
- C2, C3, C4: footprint (none) -> Capacitor_SMD:C_0805_2012Metric_Pad1.18x1.45mm_HandSolder
- D1: footprint (none) -> LED_THT:LED_D5.0mm-4_RGB_Staggered_Pins
- IC1: footprint TEENSY40 -> Flight Computer:Teensy40
- IC2: footprint XB24CAPIT-001 -> Flight Computer:XBEE_PRO_PTH
- U2: footprint KiCad:Flight-Computer_Adafruit_GPS_THT_Footprint -> Flight Computer:Adafruit_ADXL345_THT
Connections:
- net +3V3: now also D1.1 (A)
- net 12V: no longer J2.2 (Pin_2)
- net GND: now also J2.2 (Pin_2)
- net GPS-RX: now also IC1.27 (20); no longer IC1.28 (21)
- net GPS-TX: now also IC1.28 (21); no longer IC1.27 (20)
- net XBEE-RX: now also IC1.21 (14); no longer IC1.22 (15)
- net XBEE-TX: now also IC1.22 (15); no longer IC1.21 (14)
- net at D1.2 (BK): now also R4.1
- net at D1.3 (GK): now also R3.1
- net at D1.4 (RK): now also R2.1
- net Buzzer: now reaches BZ1.1 (-)
- net Buzzer: now also IC1.7 (5)
- net LED-R: now reaches IC1.4 (2)
- net LED-R: now also R2.2
- net LED-G: now reaches IC1.5 (3)
- net LED-G: now also R3.2
- net LED-B: now reaches IC1.6 (4)
- net LED-B: now also R4.2
- no-connect marks 44 -> 40
Other:
- moved on the sheet: BZ1, C1, C2, C3, C4, C5, D1, IC1, IC2, J1, J2, R1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

Commit message: Added Ignition
Parts:
- BZ1: footprint (none) -> Buzzer_Beeper:Buzzer_12x9.5RM7.6
- J1, J2: footprint (none) -> TerminalBlock:TerminalBlock_bornier-2_P5.08mm
Connections:
- net +3V3: now also BZ1.1 (-)
- net ACT2: now reaches IC1.8 (6)
- net ACT3: now reaches IC1.9 (7)
- net Buzzer renamed ACT1
- net ACT1: no longer BZ1.1 (-)
- no-connect marks 40 -> 38
Other:
- added sheet Ignition (Ignition.kicad_sch)

Commit message: Board Layout (kinda)
Parts:
- removed J1, J2: Screw_Terminal_01x02, TerminalBlock:TerminalBlock_bornier-2_P5.08mm, symbol Connector:Screw_Terminal_01x02
- added H1, H2, H3: MountingHole, MountingHole:MountingHole_2.7mm_M2.5, symbol Mechanical:MountingHole
- added J1: Screw_Terminal_01x06, TerminalBlock_4Ucon:TerminalBlock_4Ucon_1x06_P3.50mm_Horizontal, symbol Connector:Screw_Terminal_01x06
- added Q4: 2N7002, Package_TO_SOT_SMD:SOT-23, symbol Transistor_FET:2N7002
- added R7: 100, Resistor_SMD:R_0603_1608Metric_Pad0.98x0.95mm_HandSolder, symbol Device:R
- C1: value 1uf -> 10uf
- U1: value Regulator_Linear_AP2204RB-3.3 -> VXO7803-1000; footprint Package_TO_SOT_SMD:SOT-89-3 -> Package_TO_SOT_THT:TO-220-3_Horizontal_TabDown
- U2: footprint Flight Computer:Adafruit_ADXL345_THT -> Flight Computer:Adafruit_GPS_THT
Connections:
- net 12V is gone; now on net +3V3: C5.1, U1.1 (VOUT)
- net ACT3 is gone; now on net ACT2: IC1.9 (7)
- net +3V3: no longer C1.1, U1.3 (VIN)
- net ACT1: now also IC1.8 (6); no longer IC1.7 (5)
- net ACT2: no longer IC1.8 (6)
- net DROGUE_POW: now also J1.3 (Pin_3)
- net GND: now also J1.2 (Pin_2), J1.4 (Pin_4), J1.6 (Pin_6), Q4.2 (S); no longer BZ1.2 (+)
- net MAIN_POW: now also J1.5 (Pin_5)
- new net: BZ1.2 (+), Q4.3 (D)
- new net: Q4.1 (G), R7.1
- new net +BATT: C1.1, J1.1 (Pin_1), U1.3 (VIN)
- new net BUZZER: IC1.7 (5), R7.2
Other:
- sheet Ignition ports: added none; removed ACT3, AUX1_POW
- moved on the sheet: BZ1

Commit message: Finished tracing (needs optimizing)
Connections:
- net GPS-RX: now also IC1.21 (14); no longer IC1.27 (20)
- net GPS-TX: now also IC1.22 (15); no longer IC1.28 (21)
- net LED-B: now also IC1.25 (18); no longer IC1.6 (4)
- net LED-G: now also IC1.24 (17); no longer IC1.5 (3)
- net LED-R: now also IC1.23 (16); no longer IC1.4 (2)
- net XBEE-RX: now also IC1.27 (20); no longer IC1.21 (14)
- net XBEE-TX: now also IC1.28 (21); no longer IC1.22 (15)
Changed lines of the file:
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@@
   (no_connect (at 116.332 36.83))
   (no_connect (at 163.703 122.936))
-  (no_connect (at 116.332 52.07))
   (no_connect (at 71.501 181.229))
+  (no_connect (at 62.992 41.91))
   (no_connect (at 116.332 72.39))
   (no_connect (at 132.461 165.989))
@@
   (no_connect (at 71.501 183.769))
   (no_connect (at 181.737 95.631))
-  (no_connect (at 116.332 46.99))
-  (no_connect (at 116.332 49.53))
   (no_connect (at 132.461 163.449))
   (no_connect (at 132.461 176.149))
   (no_connect (at 71.501 173.609))
+  (no_connect (at 62.992 46.99))
   (no_connect (at 132.461 181.229))
+  (no_connect (at 62.992 44.45))
   (no_connect (at 71.501 171.069))
   (no_connect (at 65.913 122.428))
@@
     (stroke (width 0) (type default) (color 0 0 0 0))
   )
-  (wire (pts (xy 58.928 46.99) (xy 62.992 46.99))
-    (stroke (width 0) (type default) (color 0 0 0 0))
-  )
   (wire (pts (xy 229.616 87.122) (xy 235.839 87.122))
     (stroke (width 0) (type default) (color 0 0 0 0))
@@
     (stroke (width 0) (type default) (color 0 0 0 0))
   )
-  (wire (pts (xy 58.928 41.91) (xy 62.992 41.91))
+  (wire (pts (xy 120.396 49.53) (xy 116.332 49.53))
     (stroke (width 0) (type default) (color 0 0 0 0))
   )
@@
     (stroke (width 0) (type default) (color 0 0 0 0))
   )
+  (wire (pts (xy 120.396 52.07) (xy 116.332 52.07))
+    (stroke (width 0) (type default) (color 0 0 0 0))
+  )
   (wire (pts (xy 181.737 75.311) (xy 174.117 75.311))
     (stroke (width 0) (type default) (color 0 0 0 0))
@@
     (stroke (width 0) (type default) (color 0 0 0 0))
   )
+  (wire (pts (xy 120.396 46.99) (xy 116.332 46.99))
+    (stroke (width 0) (type default) (color 0 0 0 0))
+  )
   (wire (pts (xy 116.332 57.15) (xy 129.159 57.15))
     (stroke (width 0) (type default) (color 0 0 0 0))
@@
     (stroke (width 0) (type default) (color 0 0 0 0))
   )
-  (wire (pts (xy 58.928 44.45) (xy 62.992 44.45))
-    (stroke (width 0) (type default) (color 0 0 0 0))
-  )
   (wire (pts (xy 53.213 103.378) (xy 53.213 99.568))
     (stroke (width 0) (type default) (color 0 0 0 0))
@@
     (effects (font (size 1.27 1.27)) (justify left bottom))
   )
-  (label "XBEE-TX" (at 120.142 44.45 0)
+  (label "GPS-TX" (at 120.142 44.45 0)
     (effects (font (size 1.27 1.27)) (justify left bottom))
   )
@@
     (effects (font (size 1.27 1.27)) (justify left bottom))
   )
-  (label "GPS-TX" (at 120.904 59.69 0)
-    (effects (font (size 1.27 1.27)) (justify left bottom))
-  )
-  (label "GPS-USART" (at 146.685 62.865 0)
+  (label "XBEE-TX" (at 120.904 59.69 0)
+    (effects (font (size 1.27 1.27)) (justify left bottom))
+  )
+  (label "XBEE-USART" (at 146.304 62.738 0)
     (effects (font (size 1.27 1.27)) (justify left bottom))
   )
@@
     (effects (font (size 1.27 1.27)) (justify left bottom))
   )
-  (label "XBEE-USART" (at 145.669 47.625 0)
+  (label "GPS-USART" (at 147.066 47.498 0)
     (effects (font (size 1.27 1.27)) (justify left bottom))
   )
@@
     (effects (font (size 1.27 1.27)) (justify left bottom))
   )
-  (label "GPS-RX" (at 120.904 57.15 0)
+  (label "XBEE-RX" (at 120.904 57.15 0)
     (effects (font (size 1.27 1.27)) (justify left bottom))
   )
@@
     (effects (font (size 1.27 1.27)) (justify left bottom))
   )
-  (label "XBEE-RX" (at 120.142 41.91 0)
+  (label "GPS-RX" (at 120.142 41.91 0)
     (effects (font (size 1.27 1.27)) (justify left bottom))
   )
@@
     )
   )
-  (global_label "LED-R" (shape input) (at 58.928 41.91 180) (fields_autoplaced)
-    (effects (font (size 1.27 1.27)) (justify right))
-    (property "Intersheet References" "${INTERSHEET_REFS}" (id 0) (at 50.3143 41.8306 0)
-      (effects (font (size 1.27 1.27)) (justify right) hide)
+  (global_label "LED-G" (shape input) (at 120.396 49.53 0) (fields_autoplaced)
+    (effects (font (size 1.27 1.27)) (justify left))
+    (property "Intersheet References" "${INTERSHEET_REFS}" (id 0) (at 129.0097 49.6094 0)
+      (effects (font (size 1.27 1.27)) (justify left) hide)
+    )
+  )
+  (global_label "LED-R" (shape input) (at 120.396 46.99 0) (fields_autoplaced)
+    (effects (font (size 1.27 1.27)) (justify left))
+    (property "Intersheet References" "${INTERSHEET_REFS}" (id 0) (at 129.0097 46.9106 0)
+      (effects (font (size 1.27 1.27)) (justify left) hide)
     )
   )
@@
     )
   )
-  (global_label "LED-G" (shape input) (at 58.928 44.45 180) (fields_autoplaced)
-    (effects (font (size 1.27 1.27)) (justify right))
-    (property "Intersheet References" "${INTERSHEET_REFS}" (id 0) (at 50.3143 44.3706 0)
-      (effects (font (size 1.27 1.27)) (justify right) hide)
+  (global_label "LED-B" (shape input) (at 120.396 52.07 0) (fields_autoplaced)
+    (effects (font (size 1.27 1.27)) (justify left))
+    (property "Intersheet References" "${INTERSHEET_REFS}" (id 0) (at 129.0097 51.9906 0)
+      (effects (font (size 1.27 1.27)) (justify left) hide)
     )
   )
@@
       (effects (font (size 1.27 1.27)) (justify right) hide)
     )
-  )
-  (global_label "LED-B" (shape input) (at 58.928 46.99 180) (fields_autoplaced)
-    (effects (font (size 1.27 1.27)) (justify right))
-    (property "Intersheet References" "${INTERSHEET_REFS}" (id 0) (at 50.3143 46.9106 0)
-      (effects (font (size 1.27 1.27)) (justify right) hide)
-    )

Commit message: Fix schematic grid
Other:
- moved on the sheet: BZ1, C1, C2, C3, C4, C5, D1, H1, H2, H3, IC1, IC2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
