File: Bull Space_ Des by Sheenyl Hassan.kicad_sch (KiCad schematic)
At the start: 24 parts, among them IC1 TEENSY_4.0, IC2 XB24CZ7PIT-004, J1 Screw_Terminal_01x06, Q4 2N7002, U1 VXO7803-1000, U2 Flight-Computer_Adafruit_GPS_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, U3 ADXL343, U4 BMP280, U6 Memory_Flash_W25Q32JVSS

Commit message: Grid
Other:
- moved on the sheet: U2

Commit message: Fixed busses
Connections:
- net SCK: no longer U3.14 (SCL/SCLK), U4.4 (SCK), U6.6 (CLK)
- net ADXL-CS renamed SPI.ADXL-CS
- net BMP-CS renamed SPI.BMP-CS
- net FL-CS renamed SPI.FL-CS
- net GPS-RX renamed GPS.RX
- net GPS-TX renamed GPS.TX
- net MISO renamed SPI.MISO
- net MOSI renamed SPI.MOSI
- net XBEE-RX renamed XBEE.RX
- net XBEE-TX renamed XBEE.TX
- new net SPI.SCK: U3.14 (SCL/SCLK), U4.4 (SCK), U6.6 (CLK)
Other:
- note added: "USART"

Commit message: Power Pins Fixed (***UPDATED PCB***)
Replaced resistors and mosfet with ones from schematic.

Might want to roll back to something before this if anything goes wrong.
Connections:
- net SCK is gone; now on net SPI.SCK: IC1.20 (13)
- net +3V3: now also U2.8 (VIN); no longer U2.1 (3V3)
Changed lines of the file:
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@@
 (kicad_sch (version 20211123) (generator eeschema)
   (paper "A4")
+  (junction (at 149.86 139.7) (diameter 0) (color 0 0 0 0)
+  )
   (junction (at 59.69 74.93) (diameter 0) (color 0 0 0 0)
   )
@@
   (junction (at 30.48 163.83) (diameter 0) (color 0 0 0 0)
   )
+  (junction (at 237.49 49.53) (diameter 0) (color 0 0 0 0)
+  )
   (junction (at 243.84 146.05) (diameter 0) (color 0 0 0 0)
   )
   (junction (at 214.63 132.08) (diameter 0) (color 0 0 0 0)
-  )
-  (junction (at 237.49 49.53) (diameter 0) (color 0 0 0 0)
   )
   (junction (at 243.84 140.97) (diameter 0) (color 0 0 0 0)
@@
   (no_connect (at 62.23 39.37))
   (no_connect (at 62.23 36.83))
-  (no_connect (at 177.8 88.9))
+  (no_connect (at 177.8 71.12))
   (no_connect (at 71.12 179.07))
   (no_connect (at 132.08 171.45))
@@
     (stroke (width 0) (type default) (color 0 0 0 0))
   )
+  (wire (pts (xy 147.32 139.7) (xy 149.86 139.7))
+    (stroke (width 0) (type default) (color 0 0 0 0))
+  )
   (wire (pts (xy 40.64 22.86) (xy 40.64 64.77))
     (stroke (width 0) (type default) (color 0 0 0 0))
@@
     (stroke (width 0) (type default) (color 0 0 0 0))
   )
+  (wire (pts (xy 173.99 88.9) (xy 173.99 91.44))
+    (stroke (width 0) (type default) (color 0 0 0 0))
+  )
   (bus (pts (xy 30.48 147.32) (xy 34.29 147.32))
     (stroke (width 0) (type default) (color 0 0 0 0))
@@
     (stroke (width 0) (type default) (color 0 0 0 0))
   )
-  (wire (pts (xy 177.8 71.12) (xy 170.18 71.12))
-    (stroke (width 0) (type default) (color 0 0 0 0))
-  )
   (bus (pts (xy 24.13 54.61) (xy 24.13 57.15))
     (stroke (width 0) (type default) (color 0 0 0 0))
@@
     (stroke (width 0) (type default) (color 0 0 0 0))
   )
-  (wire (pts (xy 177.8 86.36) (xy 168.91 86.36))
-    (stroke (width 0) (type default) (color 0 0 0 0))
-  )
   (wire (pts (xy 119.38 46.99) (xy 115.57 46.99))
     (stroke (width 0) (type default) (color 0 0 0 0))
@@
     (stroke (width 0) (type default) (color 0 0 0 0))
   )
+  (wire (pts (xy 149.86 139.7) (xy 149.86 143.51))
+    (stroke (width 0) (type default) (color 0 0 0 0))
+  )
   (wire (pts (xy 246.38 135.89) (xy 243.84 135.89))
     (stroke (width 0) (type default) (color 0 0 0 0))
@@
     (stroke (width 0) (type default) (color 0 0 0 0))
   )
+  (wire (pts (xy 177.8 88.9) (xy 173.99 88.9))
+    (stroke (width 0) (type default) (color 0 0 0 0))
+  )
   (wire (pts (xy 228.6 91.44) (xy 234.95 91.44))
     (stroke (width 0) (type default) (color 0 0 0 0))
@@
     (stroke (width 0) (type default) (color 0 0 0 0))
   )
+  (wire (pts (xy 170.18 86.36) (xy 177.8 86.36))
+    (stroke (width 0) (type default) (color 0 0 0 0))
+  )
   (wire (pts (xy 119.38 74.93) (xy 124.46 74.93))
     (stroke (width 0) (type default) (color 0 0 0 0))
@@
     (stroke (width 0) (type default) (color 0 0 0 0))
   )
-  (wire (pts (xy 149.86 135.89) (xy 149.86 143.51))
+  (wire (pts (xy 149.86 135.89) (xy 149.86 139.7))
     (stroke (width 0) (type default) (color 0 0 0 0))
   )
@@
     (stroke (width 0) (type default) (color 0 0 0 0))
   )
+  (wire (pts (xy 237.49 49.53) (xy 245.11 49.53))
+    (stroke (width 0) (type default) (color 0 0 0 0))
+  )
   (wire (pts (xy 52.07 102.87) (xy 52.07 99.06))
     (stroke (width 0) (type default) (color 0 0 0 0))
@@
     (stroke (width 0) (type default) (color 0 0 0 0))
   )
-  (wire (pts (xy 237.49 49.53) (xy 245.11 49.53))
-    (stroke (width 0) (type default) (color 0 0 0 0))
-  )
   (wire (pts (xy 115.57 59.69) (xy 128.27 59.69))
     (stroke (width 0) (type default) (color 0 0 0 0))
@@
     (stroke (width 0) (type default) (color 0 0 0 0))
   )
+  (wire (pts (xy 170.18 90.17) (xy 170.18 86.36))
+    (stroke (width 0) (type default) (color 0 0 0 0))
+  )
   (wire (pts (xy 217.17 132.08) (xy 214.63 132.08))
     (stroke (width 0) (type default) (color 0 0 0 0))
@@
     (effects (font (size 1.27 1.27)) (justify left bottom))
   )
-  (label "SCK" (at 121.539 39.37 0)
+  (label "SPI.SCK" (at 119.38 39.37 0)
     (effects (font (size 1.27 1.27)) (justify left bottom))
   )
@@
     (pin "1")
   )
-  (symbol (lib_id "power:GND") (at 168.91 86.36 0) (unit 1)
-    (in_bom yes) (on_board yes)
-    (property "Reference" "#PWR0107" (id 0) (at 168.91 92.71 0)
-      (effects (font (size 1.27 1.27)) hide)
-    )
-    (property "Value" "GND" (id 1) (at 169.037 89.6112 90)
+  (symbol (lib_id "power:GND") (at 170.18 90.17 0) (unit 1)
+    (in_bom yes) (on_board yes)
+    (property "Reference" "#PWR0107" (id 0) (at 170.18 96.52 0)
+      (effects (font (size 1.27 1.27)) hide)
+    )
+    (property "Value" "GND" (id 1) (at 170.307 93.4212 90)
       (effects (font (size 1.27 1.27)) (justify right))
     )
-    (property "Footprint" "" (id 2) (at 168.91 86.36 0)
-      (effects (font (size 1.27 1.27)) hide)
-    )
-    (property "Datasheet" "" (id 3) (at 168.91 86.36 0)
+    (property "Footprint" "" (id 2) (at 170.18 90.17 0)
+      (effects (font (size 1.27 1.27)) hide)
+    )
+    (property "Datasheet" "" (id 3) (at 170.18 90.17 0)
       (effects (font (size 1.27 1.27)) hide)
     )
@@
     (pin "1")
   )
+  (symbol (lib_id "power:PWR_FLAG") (at 237.49 49.53 0) (unit 1)
+    (in_bom yes) (on_board yes) (fields_autoplaced)
+    (property "Reference" "#FLG0101" (id 0) (at 237.49 47.625 0)
+      (effects (font (size 1.27 1.27)) hide)
+    )
+    (property "Value" "PWR_FLAG" (id 1) (at 237.49 44.45 0))
+    (property "Footprint" "" (id 2) (at 237.49 49.53 0)
+      (effects (font (size 1.27 1.27)) hide)
+    )
+    (property "Datasheet" "~" (id 3) (at 237.49 49.53 0)
+      (effects (font (size 1.27 1.27)) hide)
+    )
+    (pin "1")
+  )
   (symbol (lib_id "power:+3.3V") (at 123.19 67.31 270) (unit 1)
     (in_bom yes) (on_board yes) (fields_autoplaced)
@@
     )
     (property "Datasheet" "" (id 3) (at 264.16 100.33 0)
+      (effects (font (size 1.27 1.27)) hide)
+    )
+    (pin "1")
+  )
+  (symbol (lib_id "power:PWR_FLAG") (at 147.32 139.7 90) (unit 1)
+    (in_bom yes) (on_board yes) (fields_autoplaced)
+    (property "Reference" "#FLG0102" (id 0) (at 145.415 139.7 0)
+      (effects (font (size 1.27 1.27)) hide)
+    )
+    (property "Value" "PWR_FLAG" (id 1) (at 143.51 139.6999 90)
+      (effects (font (size 1.27 1.27)) (justify left))
+    )
+    (property "Footprint" "" (id 2) (at 147.32 139.7 0)
+      (effects (font (size 1.27 1.27)) hide)
+    )
+    (property "Datasheet" "~" (id 3) (at 147.32 139.7 0)
       (effects (font (size 1.27 1.27)) hide)
     )
@@
     (pin "6")
   )
-  (symbol (lib_id "power:+3.3V") (at 170.18 71.12 90) (unit 1)
-    (in_bom yes) (on_board yes) (fields_autoplaced)
-    (property "Reference" "#PWR0118" (id 0) (at 173.99 71.12 0)
-      (effects (font (size 1.27 1.27)) hide)
-    )
-    (property "Value" "+3.3V" (id 1) (at 165.862 71.1201 90)
-      (effects (font (size 1.27 1.27)) (justify left))
-    )
-    (property "Footprint" "" (id 2) (at 170.18 71.12 0)
-      (effects (font (size 1.27 1.27)) hide)
-    )
-    (property "Datasheet" "" (id 3) (at 170.18 71.12 0)
+  (symbol (lib_id "power:+3.3V") (at 173.99 91.44 180) (unit 1)
+    (in_bom yes) (on_board yes)
+    (property "Reference" "#PWR0118" (id 0) (at 173.99 87.63 0)
+      (effects (font (size 1.27 1.27)) hide)
+    )
+    (property "Value" "+3.3V" (id 1) (at 173.99 93.98 90)
+      (effects (font (size 1.27 1.27)) (justify left))
+    )
+    (property "Footprint" "" (id 2) (at 173.99 91.44 0)
+      (effects (font (size 1.27 1.27)) hide)
+    )
+    (property "Datasheet" "" (id 3) (at 173.99 91.44 0)
       (effects (font (size 1.27 1.27)) hide)
     )
@@
   )
   (symbol_instances
+    (path "/24262ee6-ead1-4117-9935-992cab39ff81"
+      (reference "#FLG0101") (unit 1) (value "PWR_FLAG") (footprint "")
+    )
+    (path "/4442bca2-41c2-4775-869a-4d6c8c1a9fef"
+      (reference "#FLG0102") (unit 1) (value "PWR_FLAG") (footprint "")
+    )
     (path "/e9edb235-fe63-4090-aec0-86a4c7615d5d/00000000-0000-0000-0000-00005c0747de"
       (reference "#PWR027") (unit 1) (value "+BATT") (footprint "")
